File: schematic/buttler_pcb.kicad_pcb (KiCad board)
At the start: 2 copper layers, 50.8 x 35.6 mm, 12 parts, among them J1 HL, J2 HR, J3 ISP, J4 RF Receiver, J5 IO, J6 ISP 2, U1 PC817, U2 PC817, U3 PC817

Commit message: Repo Sync
Parts:
- added C1: 100nF, Capacitor_SMD:C_0402_1005Metric, F.Cu at (155.1, 61.0)
- added C2: 100nF, Capacitor_SMD:C_0402_1005Metric, F.Cu at (135.9, 61.0)
- added D1: LED, LED_SMD:LED_0603_1608Metric, F.Cu at (121.2, 78.5)
- added D2: LED, LED_SMD:LED_0603_1608Metric, F.Cu at (122.9, 78.5)
- added D3: LED, LED_SMD:LED_0603_1608Metric, F.Cu at (124.7, 78.5)
- added D4: LED, LED_SMD:LED_0603_1608Metric, F.Cu at (126.5, 78.5)
- added R4: 330r, Resistor_SMD:R_0603_1608Metric, F.Cu at (121.2, 75.2)
- added R5: 330r, Resistor_SMD:R_0603_1608Metric, F.Cu at (122.9, 75.2)
- added R6: 330r, Resistor_SMD:R_0603_1608Metric, F.Cu at (124.7, 75.2)
- added R7: 330r, Resistor_SMD:R_0603_1608Metric, F.Cu at (126.5, 75.2)
- added SW1: Reset, Button_Switch_SMD:SW_SPST_TL3342, F.Cu at (151.9, 56.6)
- added SW2: Pgm/Factory, Button_Switch_SMD:SW_SPST_TL3342, F.Cu at (141.5, 56.6)
- J1, J2, J3, J5: moved to F.Cu
- R1, R2, R3: footprint Resistor_THT:R_Axial_DIN0204_L3.6mm_D1.6mm_P2.54mm_Vertical -> Resistor_SMD:R_0603_1608Metric
- U1, U2, U3: footprint Package_DIP:DIP-4_W7.62mm -> Package_SO:SOP-4_3.8x4.1mm_P2.54mm
- moved J4 80.3 mm to (125.5, 50.8)
- moved U1 78.0 mm to (138.4, 66.0)
- moved U2 70.0 mm to (144.8, 65.8)
- moved U3 63.9 mm to (151.1, 65.8)
- moved J6 52.2 mm to (144.8, 47.5), turned to 90 degrees
- moved J1 33.0 mm to (129.5, 50.8), turned to 0 degrees
- moved R3 29.1 mm to (150.7, 71.1)
- moved J2 27.9 mm to (160.0, 50.8), turned to 0 degrees
- moved R2 25.1 mm to (145.2, 71.1)
- moved R1 23.4 mm to (138.9, 71.1)
- moved J3 12.7 mm to (139.7, 50.8)
- moved J5 11.5 mm to (138.4, 77.5), turned to 0 degrees
Connections:
- J1 pad 12: unconnected-(J1-Pin_12-Pad12) -> STATUS_LED
- J1 pad 13: unconnected-(J1-Pin_13-Pad13) -> ENDSTOP_O_LED
- J1 pad 14: unconnected-(J1-Pin_14-Pad14) -> GNDREF
- J1 pad 15: unconnected-(J1-Pin_15-Pad15) -> ENDSTOP_C_LED
- J1 pad 18: unconnected-(J1-Pin_18-Pad18) -> BARRIER_LED
- J1 pad 20: unconnected-(J1-Pin_20-Pad20) -> GNDREF
- J1 pad 7: unconnected-(J1-Pin_7-Pad7) -> PGM
- J2 pad 17: unconnected-(J2-Pin_17-Pad17) -> EN
- J2 pad 2: unconnected-(J2-Pin_2-Pad2) -> GNDREF
- J3 pad 6: Net-(J3-Pin_6) -> +5V
- J6 pad 4: Net-(J3-Pin_6) -> +5V
Routing:
- net GNDREF: track 0.00 -> 52.9 mm
- net DATA: track 0.00 -> 52.1 mm, vias 1 -> 0
- net GND: track 0.00 -> 34.5 mm
- net ENDSTOP_O_LED: track 0.00 -> 29.9 mm, vias 0 -> 2
- net STATUS_LED: track 0.00 -> 28.5 mm
- net EN: track 0.00 -> 23.6 mm
- net ENDSTOP_OPEN: track 0.00 -> 21.2 mm
- net PGM: track 0.00 -> 18.7 mm
- net +5V: track 0.00 -> 18.5 mm
- net ENDSTOP_C_LED: track 0.00 -> 17.3 mm, vias 0 -> 1
- net BARRIER_LED: track 0.00 -> 16.8 mm
- net ENDSTOP_CLOSED: track 0.00 -> 13.4 mm
- net Net-(J5-Pin_2): track 0.00 -> 9.42 mm
- net Net-(J5-Pin_3): track 0.00 -> 8.07 mm
- net Net-(J5-Pin_4): track 0.00 -> 7.77 mm
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- added copper zone on F.Cu, net +5V
- added copper zone on B.Cu, net GNDREF
Other:
- outline, holes or cut-outs redrawn

Commit message: Repo Sync
Parts:
- added RF1: ~, buttler:RXB12, F.Cu at (117.1, 61.7)
- J4: value RF Receiver -> IPEX; footprint Connector_PinHeader_2.54mm:PinHeader_1x04_P2.54mm_Vertical -> buttler:IPEX_20279-001E-03
- moved J4 1.11 mm to (125.0, 49.8), turned to 180 degrees
Connections:
- J4 pad 1: +5V -> Net-(J4-Pin_1)
- J4 pad 2: DATA -> Net-(J4-Pin_2)
Routing:
- net Net-(J4-Pin_2): track 0.00 -> 13.8 mm
- net +5V: track 18.5 -> 5.42 mm
- net Net-(J4-Pin_1): track 0.00 -> 11.4 mm
- net DATA: track 52.1 -> 60.5 mm

Commit message: Repo Sync
Parts:
- U1, U2, U3: footprint Package_SO:SOP-4_3.8x4.1mm_P2.54mm -> schematic:OPTO-SMD4
- moved C1 3.18 mm to (157.1, 58.5), turned to 0 degrees
- moved R3 2.58 mm to (153.0, 72.2)
- moved C2 2.47 mm to (135.5, 58.5), turned to 0 degrees
- moved U3 2.29 mm to (153.4, 65.8), turned to 0 degrees
- moved U2 1.52 mm to (146.3, 65.8), turned to 0 degrees
- moved R2 1.52 mm to (146.3, 72.2)
- moved R1 1.19 mm to (139.1, 72.3)
- moved U1 0.73 mm to (139.1, 65.7), turned to 0 degrees
- moved SW1 0.63 mm to (151.3, 56.6)
Routing:
- net GNDREF: track 52.9 -> 85.5 mm, vias 3 -> 2
- net ENDSTOP_OPEN: track 21.2 -> 23.9 mm, vias 1 -> 0
- net Net-(J5-Pin_4): track 7.77 -> 5.30 mm
- net Net-(J5-Pin_3): track 8.07 -> 5.91 mm
- net Net-(J5-Pin_2): track 9.42 -> 7.97 mm
- net GND: track 34.5 -> 35.9 mm
- net PGM: track 18.7 -> 17.6 mm
- net Net-(R2-Pad2): track 2.91 -> 2.12 mm
- net ENDSTOP_CLOSED: track 13.4 -> 14.1 mm, vias 1 -> 0
- net EN: track 23.6 -> 24.3 mm, vias 0 -> 1
- net Net-(R3-Pad2): track 2.54 -> 1.97 mm
Other:
- board text added: "+"
- board text added: "-"
- board text added: "5V"
- board text added: "BAR"
- board text added: "COM"
- board text added: "ESC"
- board text added: "ESO"
- board text added: "Gnd"
- board text added: "IO0"
- board text added: "Rui Barreiros 2024 Rev 1 ESP32 Relay X1 v1.2 Hat"
- board text added: "Rx"
- board text added: "Tx"
